File: project/project.kicad_sch (KiCad schematic)
At the start: 40 parts, among them J1 TYPE-C-31-M-12, J2 IDC EDGE 2x8, Q1 DTC114YUA, Q2 DTC114YUA, SW1 RESET, SW2 ESP Power, U1 USBLC6-2SC6, U2 ME6211C33M5G-N, U3 CH340C

Commit message: adding mating connector to bom
Parts:
- added J3: IDC HEADER 2x8, symbol Connector_Generic:Conn_02x08_Odd_Even
Connections:
- no-connect marks 16 -> 32
Other:
- note added: "Mating connector for BOM"
- title: esp-12f-flasher/USB-UART -> esp-flasher
Changed lines of the file:
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@@
   (paper "A4")
   (title_block
-    (title "esp-12f-flasher/USB-UART")
-    (date "2023-02-12")
+    (title "esp-flasher")
+    (date "2023-02-16")
     (rev "2.0")
     (company "makerspace.lt")
@@
   (junction (at 88.9 81.28) (diameter 0) (color 0 0 0 0)
   )
+  (no_connect (at 81.28 171.45))
   (no_connect (at 144.78 73.66))
+  (no_connect (at 78.74 184.15))
+  (no_connect (at 78.74 171.45))
   (no_connect (at 165.1 86.36))
+  (no_connect (at 73.66 171.45))
+  (no_connect (at 88.9 171.45))
   (no_connect (at 158.75 135.89))
+  (no_connect (at 71.12 184.15))
   (no_connect (at 165.1 83.82))
   (no_connect (at 165.1 78.74))
+  (no_connect (at 71.12 171.45))
   (no_connect (at 88.9 91.44))
   (no_connect (at 88.9 88.9))
   (no_connect (at 146.05 143.51))
   (no_connect (at 146.05 133.35))
+  (no_connect (at 86.36 184.15))
+  (no_connect (at 83.82 184.15))
+  (no_connect (at 81.28 184.15))
   (no_connect (at 165.1 81.28))
+  (no_connect (at 83.82 171.45))
+  (no_connect (at 86.36 171.45))
   (no_connect (at 146.05 140.97))
+  (no_connect (at 76.2 184.15))
+  (no_connect (at 76.2 171.45))
+  (no_connect (at 88.9 184.15))
   (no_connect (at 134.62 40.64))
   (no_connect (at 146.05 146.05))
@@
   (no_connect (at 158.75 138.43))
   (no_connect (at 66.04 99.06))
+  (no_connect (at 73.66 184.15))
   (wire (pts (xy 110.49 134.62) (xy 110.49 127))
     (stroke (width 0) (type default) (color 0 0 0 0))
@@
     (stroke (width 0) (type default) (color 0 0 0 0))
   )
+  (polyline (pts (xy 129.54 190.5) (xy 50.8 190.5))
+    (stroke (width 0) (type solid) (color 0 0 0 0))
+  )
   (polyline (pts (xy 241.3 109.22) (xy 241.3 160.02))
     (stroke (width 0) (type solid) (color 0 0 0 0))
@@
     (stroke (width 0) (type default) (color 0 0 0 0))
   )
+  (polyline (pts (xy 129.54 160.02) (xy 129.54 190.5))
+    (stroke (width 0) (type solid) (color 0 0 0 0))
+  )
   (wire (pts (xy 88.9 68.58) (xy 99.06 68.58))
     (stroke (width 0) (type default) (color 0 0 0 0))
@@
   (wire (pts (xy 194.31 82.55) (xy 193.04 82.55))
     (stroke (width 0) (type default) (color 0 0 0 0))
+  )
+  (polyline (pts (xy 50.8 160.02) (xy 50.8 190.5))
+    (stroke (width 0) (type solid) (color 0 0 0 0))
   )
   (wire (pts (xy 153.67 57.15) (xy 158.75 57.15))
@@
   )
   (text "ESP pull-ups" (at 52.07 114.3 0)
+    (effects (font (size 3 3)) (justify left bottom))
+  )
+  (text "Mating connector for BOM" (at 52.07 165.1 0)
     (effects (font (size 3 3)) (justify left bottom))
   )
@@
     (pin "6")
   )
-  (symbol (lib_id "power:GND") (at 273.05 158.75 0) (unit 1)
-    (in_bom yes) (on_board yes)
-    (property "Reference" "#PWR023" (id 0) (at 273.05 165.1 0)
-      (effects (font (size 1.27 1.27)) hide)
-    )
-    (property "Value" "GND" (id 1) (at 273.05 162.56 0)
-      (effects (font (size 1.27 1.27)) hide)
-    )
-    (property "Footprint" "" (id 2) (at 273.05 158.75 0)
-      (effects (font (size 1.27 1.27)) hide)
-    )
-    (property "Datasheet" "" (id 3) (at 273.05 158.75 0)
+  (symbol (lib_id "power:GND") (at 165.1 180.34 0) (unit 1)
+    (in_bom yes) (on_board yes)
+    (property "Reference" "#PWR023" (id 0) (at 165.1 186.69 0)
+      (effects (font (size 1.27 1.27)) hide)
+    )
+    (property "Value" "GND" (id 1) (at 165.1 184.15 0)
+      (effects (font (size 1.27 1.27)) hide)
+    )
+    (property "Footprint" "" (id 2) (at 165.1 180.34 0)
+      (effects (font (size 1.27 1.27)) hide)
+    )
+    (property "Datasheet" "" (id 3) (at 165.1 180.34 0)
       (effects (font (size 1.27 1.27)) hide)
     )
@@
     (pin "2")
   )
-  (symbol (lib_id "power:PWR_FLAG") (at 273.05 158.75 0) (unit 1)
+  (symbol (lib_id "power:PWR_FLAG") (at 165.1 180.34 0) (unit 1)
     (in_bom yes) (on_board yes) (fields_autoplaced)
-    (property "Reference" "#FLG02" (id 0) (at 273.05 156.845 0)
-      (effects (font (size 1.27 1.27)) hide)
-    )
-    (property "Value" "PWR_FLAG" (id 1) (at 273.05 153.67 0))
-    (property "Footprint" "" (id 2) (at 273.05 158.75 0)
-      (effects (font (size 1.27 1.27)) hide)
-    )
-    (property "Datasheet" "~" (id 3) (at 273.05 158.75 0)
+    (property "Reference" "#FLG02" (id 0) (at 165.1 178.435 0)
+      (effects (font (size 1.27 1.27)) hide)
+    )
+    (property "Value" "PWR_FLAG" (id 1) (at 165.1 175.26 0))
+    (property "Footprint" "" (id 2) (at 165.1 180.34 0)
+      (effects (font (size 1.27 1.27)) hide)
+    )
+    (property "Datasheet" "~" (id 3) (at 165.1 180.34 0)
       (effects (font (size 1.27 1.27)) hide)
     )
@@
     (pin "2")
   )
-  (symbol (lib_id "-local:LOGO_KMS") (at 161.29 181.61 0) (unit 1)
+  (symbol (lib_id "-local:LOGO_KMS") (at 262.89 31.75 0) (unit 1)
     (in_bom no) (on_board yes) (fields_autoplaced)
-    (property "Reference" "G2" (id 0) (at 161.29 167.6823 0)
-      (effects (font (size 1.27 1.27)) hide)
-    )
-    (property "Value" "LOGO_KMS" (id 1) (at 161.29 195.5377 0)
-      (effects (font (size 1.27 1.27)) hide)
-    )
-    (property "Footprint" "-local:logo_kms_small_silkscreen" (id 2) (at 161.29 181.61 0)
-      (effects (font (size 1.27 1.27)) hide)
-    )
-    (property "Datasheet" "" (id 3) (at 161.29 181.61 0)
+    (property "Reference" "G2" (id 0) (at 262.89 17.8223 0)
+      (effects (font (size 1.27 1.27)) hide)
+    )
+    (property "Value" "LOGO_KMS" (id 1) (at 262.89 45.6777 0)
+      (effects (font (size 1.27 1.27)) hide)
+    )
+    (property "Footprint" "-local:logo_kms_small_silkscreen" (id 2) (at 262.89 31.75 0)
+      (effects (font (size 1.27 1.27)) hide)
+    )
+    (property "Datasheet" "" (id 3) (at 262.89 31.75 0)
       (effects (font (size 1.27 1.27)) hide)
     )
@@
     (pin "2")
   )
+  (symbol (lib_id "Connector_Generic:Conn_02x08_Odd_Even") (at 78.74 179.07 90) (unit 1)
+    (in_bom yes) (on_board no)
+    (property "Reference" "J3" (id 0) (at 93.98 175.26 90)
+      (effects (font (size 1.27 1.27)) (justify left))
+    )
+    (property "Value" "IDC HEADER 2x8" (id 1) (at 107.95 179.07 90)
+      (effects (font (size 1.27 1.27)) (justify left))
+    )
+    (property "Footprint" "" (id 2) (at 78.74 179.07 0)
+      (effects (font (size 1.27 1.27)) hide)
+    )
+    (property "Datasheet" "~" (id 3) (at 78.74 179.07 0)
+      (effects (font (size 1.27 1.27)) hide)
+    )
+    (property "jlc-part-type" "-" (id 4) (at 78.74 179.07 0)
+      (effects (font (size 1.27 1.27)) hide)
+    )
+    (property "lcsc#" "C3406" (id 5) (at 78.74 179.07 0)
+      (effects (font (size 1.27 1.27)) hide)
+    )
+    (pin "1")
+    (pin "10")
+    (pin "11")
+    (pin "12")
+    (pin "13")
+    (pin "14")
+    (pin "15")
+    (pin "16")
+    (pin "2")
+    (pin "3")
+    (pin "4")
+    (pin "5")
+    (pin "6")
+    (pin "7")
+    (pin "8")
+    (pin "9")
+  )
   (symbol (lib_id "power:GND") (at 140.97 48.26 0) (unit 1)
     (in_bom yes) (on_board yes)
@@
     (pin "5")
   )
-  (symbol (lib_id "Graphic:Logo_Open_Hardware_Large") (at 132.08 181.61 0) (unit 1)
+  (symbol (lib_id "Graphic:Logo_Open_Hardware_Large") (at 30.48 30.48 0) (unit 1)
     (in_bom no) (on_board yes) (fields_autoplaced)
-    (property "Reference" "G1" (id 0) (at 132.08 168.91 0)
-      (effects (font (size 1.27 1.27)) hide)
-    )
-    (property "Value" "Logo_Open_Hardware_Large" (id 1) (at 132.08 191.77 0)
-      (effects (font (size 1.27 1.27)) hide)
-    )
-    (property "Footprint" "Symbol:OSHW-Symbol_6.7x6mm_SilkScreen" (id 2) (at 132.08 181.61 0)
-      (effects (font (size 1.27 1.27)) hide)
-    )
-    (property "Datasheet" "~" (id 3) (at 132.08 181.61 0)
+    (property "Reference" "G1" (id 0) (at 30.48 17.78 0)
+      (effects (font (size 1.27 1.27)) hide)
+    )
+    (property "Value" "Logo_Open_Hardware_Large" (id 1) (at 30.48 40.64 0)
+      (effects (font (size 1.27 1.27)) hide)
+    )
+    (property "Footprint" "Symbol:OSHW-Symbol_6.7x6mm_SilkScreen" (id 2) (at 30.48 30.48 0)
+      (effects (font (size 1.27 1.27)) hide)
+    )
+    (property "Datasheet" "~" (id 3) (at 30.48 30.48 0)
       (effects (font (size 1.27 1.27)) hide)
     )
@@
       (reference "J2") (unit 1) (value "IDC EDGE 2x8") (footprint "-local:IDC-Female_2x08_P2.54mm_Edge")
     )
+    (path "/7d815bf5-f282-4b65-a62e-540131db0a6d"
+      (reference "J3") (unit 1) (value "IDC HEADER 2x8") (footprint "")
+    )
     (path "/8f41fdf4-190a-4a65-88a4-0092446ec00a"

Commit message: making leds colorful
Parts:
- removed J3: IDC HEADER 2x8, symbol Connector_Generic:Conn_02x08_Odd_Even
- added J3: matching connector for BOM, symbol Connector_Generic:Conn_01x01
- G1, G2: jlc-part-type (none) -> -
- LED1: value PWR -> PWR-yellow; jlc-part-type B -> E; lcsc# C2297 -> C779458
- LED2: value TX -> TX-blue; jlc-part-type B -> E; lcsc# C2297 -> C965817
- LED3: value RX -> RX-green; jlc-part-type B -> E; lcsc# C2297 -> C965815
- LED4: value ESP -> ESP-red; lcsc# C2297 -> C84256
Connections:
- no-connect marks 32 -> 17
Other:
- note removed: "Mating connector for BOM"
